File: Issue1/ZX26_Computer_CPU_ULA.kicad_sch (KiCad schematic)
At the start: 45 parts, among them J4 VIDEO OUT, J5 TAPE IN, J6 TAPE OUT, Q1 2N3904, Q2 2N3904, SW42 USA/UK, U1 vLA81 ULA, U3 Z80 CPU

Commit message: Minor PCB updates
Parts:
- J5: value TAPE IN -> TAPE IN (EAR)
- J6: value TAPE OUT -> TAPE OUT (MIC)
Changed lines of the file:
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@@
 			)
 		)
-		(property "Value" "TAPE OUT"
+		(property "Value" "TAPE OUT (MIC)"
 			(at 30.734 64.516 0)
 			(show_name no)
@@
 			)
 		)
-		(property "Value" "TAPE IN"
+		(property "Value" "TAPE IN (EAR)"
 			(at 53.34 112.3949 0)
 			(show_name no)
