File: Issue1/ZX26_Computer_Memory.kicad_sch (KiCad schematic)
At the start: 3 parts, among them SW41 ROM BANK SELECT, U2 62256 32KB RAM, U4 27C256 32KB ROM

Commit message: Minor PCB updates
Changed lines of the file:
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@@
+		)
+	)
+	(text_box "vLA81 SW3/SW4 RAM Settings\nMODE 0 (ON/OFF): 16KB (4000-7FFF) [STANDARD ZX81]\nMODE 1 (OFF/ON): 32KB (4000-BFFF) [UPPER 32KB HIRES]\nMODE 2 (OFF/ON): 32KB (2000-9FFF) [LOWER 32KB WRX HIRES]\nMODE 3  (ON/ON): 32KB (0000-7FFF) [SOFT CONFIG]"
+		(exclude_from_sim no)
+		(at 38.1 41.91 0)
+		(size 67.31 12.7)
+		(margins 0.9525 0.9525 0.9525 0.9525)
+		(stroke
+			(width 0)
+			(type solid)
+		)
+		(fill
+			(type none)
+		)
+		(effects
+			(font
+				(size 1.27 1.27)
+			)
+			(justify left top)
 		)
 	)
