File: Issue1/ZX26_Computer.kicad_pcb (KiCad board)
At the start: 2 copper layers, 262.5 x 140.5 mm, 125 parts, among them J1 USB POWER IN, J2 ATARI JOYSTICK, J3 SPACE/0, J4 VIDEO OUT, J5 TAPE IN, J6 TAPE OUT, Q1 2N3904, Q2 2N3904, Q3 2N3904, Q4 2N3904, Q5 2N3904, Q6 2N3904, Q7 2N3904, Q8 2N3904, SW1 1, SW10 E, SW11 D, SW12 X, SW13 4, SW14 R, SW15 F, SW16 C, SW17 5, SW18 T, SW19 G, SW2 Q, SW20 V, SW21 6, SW22 Y, SW23 H, SW24 B, SW25 7, SW26 U, SW27 J, SW28 N, SW29 8, SW3 A, SW30 I, SW31 K, SW32 M, SW33 9, SW34 O, SW35 L, SW36 DOT, SW37 ZERO, SW38 P, SW39 NL, SW4 SHIFT, SW40 SPACE, SW41 ROM BANK SELECT, SW42 USA/UK, SW43 LEFT, SW44 DOWN, SW45 UP, SW46 RIGHT, SW5 2, SW6 W, SW7 S, SW8 Z, SW9 3, U1 vLA81 ULA, U2 62256 32KB RAM, U3 Z80 CPU, U4 27C256 32KB ROM

Commit message: Minor PCB updates
Parts:
- J5: value TAPE IN -> TAPE IN (EAR)
- J6: value TAPE OUT -> TAPE OUT (MIC)
Connections:
- net ~{NMI} renamed /ZX26 CPU & ULA/~{NMI}
Routing:
- net GND: track 376.8 -> 367.5 mm
- net D7': track 76.2 -> 69.0 mm
- net D6': track 71.1 -> 64.8 mm
- net Net-(U1-A6'): track 86.5 -> 81.0 mm
- net D1': track 64.0 -> 58.6 mm
- net D2': track 59.1 -> 53.8 mm
- net D5': track 65.8 -> 60.7 mm
- net D0': track 68.1 -> 63.4 mm
- net A10: track 148.1 -> 144.4 mm
- net D4': track 60.4 -> 58.4 mm
- net D3': track 58.8 -> 57.8 mm
- net Net-(U1-A8'): track 96.8 -> 95.9 mm, vias 0 -> 1
- net Net-(U1-A7'): vias 0 -> 1

Commit message: Additional PCB text
Parts:
- J3: value SPACE/0 -> FIRE MAPPING
Other:
- board text added: "SPACE"
- board text added: "ZERO"
Changed lines of the file:
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@@
 			)
 		)
-		(property "Value" "SPACE/0"
-			(at 0 7.46 0)
+		(property "Value" "FIRE MAPPING"
+			(at -0.635 7.46 0)
 			(layer "F.SilkS")
 			(effects
@@
 		(layer "Edge.Cuts")
 	)
+	(gr_text "SPACE"
+		(at 292.9046 121.74697 0)
+		(layer "F.SilkS")
+		(effects
+			(font
+				(size 1 1)
+				(thickness 0.1)
+			)
+			(justify left bottom)
+		)
+	)
+	(gr_text "ZERO"
+		(at 292.9046 126.82697 0)
+		(layer "F.SilkS")
+		(effects
+			(font
+				(size 1 1)
+				(thickness 0.1)
+			)
+			(justify left bottom)
+		)
+	)
 	(gr_text "ISSUE 1"
 		(at 259.8846 69.67697 0)
@@
 	)
 	(segment
+		(start 110.406 97.94197)
+		(end 101.1996 97.94197)
+		(width 0.2)
+		(layer "F.Cu")
+		(net "/ZX26 CPU & ULA/~{NMI}")
+	)
+	(segment
+		(start 110.6538 97.69417)
+		(end 110.406 97.94197)
+		(width 0.2)
+		(layer "F.Cu")
+		(net "/ZX26 CPU & ULA/~{NMI}")
+	)
+	(via
+		(at 110.6538 97.69417)
+		(size 0.6)
+		(drill 0.3)
+		(layers "F.Cu" "B.Cu")
+		(net "/ZX26 CPU & ULA/~{NMI}")
+	)
+	(segment
+		(start 124.8408 96.52577)
+		(end 111.8222 96.52577)
+		(width 0.2)
+		(layer "B.Cu")
+		(net "/ZX26 CPU & ULA/~{NMI}")
+	)
+	(segment
+		(start 125.3296 96.03697)
+		(end 130.1796 100.88697)
+		(width 0.2)
+		(layer "B.Cu")
+		(net "/ZX26 CPU & ULA/~{NMI}")
+	)
+	(segment
+		(start 111.8222 96.52577)
+		(end 110.6538 97.69417)
+		(width 0.2)
+		(layer "B.Cu")
+		(net "/ZX26 CPU & ULA/~{NMI}")
+	)
+	(segment
+		(start 136.8896 100.88697)
+		(end 139.0246 103.02197)
+		(width 0.2)
+		(layer "B.Cu")
+		(net "/ZX26 CPU & ULA/~{NMI}")
+	)
+	(segment
+		(start 130.1796 100.88697)
+		(end 136.8896 100.88697)
+		(width 0.2)
+		(layer "B.Cu")
+		(net "/ZX26 CPU & ULA/~{NMI}")
+	)
+	(segment
+		(start 125.3296 96.03697)
+		(end 124.8408 96.52577)
+		(width 0.2)
+		(layer "B.Cu")
+		(net "/ZX26 CPU & ULA/~{NMI}")
+	)
+	(segment
 		(start 124.6046 99.21197)
 		(end 123.4246 99.21197)
@@
 		(net "Net-(U1-A5')")
 	)
-	(segment
-		(start 110.406 97.94197)
-		(end 101.1996 97.94197)
-		(width 0.2)
-		(layer "F.Cu")
-		(net "/ZX26 CPU & ULA/~{NMI}")
-	)
-	(segment
-		(start 110.6538 97.69417)
-		(end 110.406 97.94197)
-		(width 0.2)
-		(layer "F.Cu")
-		(net "/ZX26 CPU & ULA/~{NMI}")
-	)
-	(via
-		(at 110.6538 97.69417)
-		(size 0.6)
-		(drill 0.3)
-		(layers "F.Cu" "B.Cu")
-		(net "/ZX26 CPU & ULA/~{NMI}")
-	)
-	(segment
-		(start 124.8408 96.52577)
-		(end 111.8222 96.52577)
-		(width 0.2)
-		(layer "B.Cu")
-		(net "/ZX26 CPU & ULA/~{NMI}")
-	)
-	(segment
-		(start 125.3296 96.03697)
-		(end 130.1796 100.88697)
-		(width 0.2)
-		(layer "B.Cu")
-		(net "/ZX26 CPU & ULA/~{NMI}")
-	)
-	(segment
-		(start 111.8222 96.52577)
-		(end 110.6538 97.69417)
-		(width 0.2)
-		(layer "B.Cu")
-		(net "/ZX26 CPU & ULA/~{NMI}")
-	)
-	(segment
-		(start 136.8896 100.88697)
-		(end 139.0246 103.02197)
-		(width 0.2)
-		(layer "B.Cu")
-		(net "/ZX26 CPU & ULA/~{NMI}")
-	)
-	(segment
-		(start 130.1796 100.88697)
-		(end 136.8896 100.88697)
-		(width 0.2)
-		(layer "B.Cu")
-		(net "/ZX26 CPU & ULA/~{NMI}")
-	)
-	(segment
-		(start 125.3296 96.03697)
-		(end 124.8408 96.52577)
-		(width 0.2)
-		(layer "B.Cu")
-		(net "/ZX26 CPU & ULA/~{NMI}")
-	)
 	(zone
