File: Issue1/ZX26_Computer_Keyboard_Joystick.kicad_sch (KiCad schematic)
At the start: 68 parts, among them J2 ATARI JOYSTICK, J3 SPACE/0, Q3 2N3904, Q4 2N3904, Q5 2N3904, Q6 2N3904, Q7 2N3904, Q8 2N3904, SW1 1, SW10 E, SW11 D, SW12 X, SW13 4, SW14 R, SW15 F, SW16 C, SW17 5, SW18 T, SW19 G, SW2 Q, SW20 V, SW21 6, SW22 Y, SW23 H, SW24 B, SW25 7, SW26 U, SW27 J, SW28 N, SW29 8, SW3 A, SW30 I, SW31 K, SW32 M, SW33 9, SW34 O, SW35 L, SW36 DOT, SW37 ZERO, SW38 P, SW39 NL, SW4 SHIFT, SW40 SPACE, SW43 LEFT, SW44 DOWN, SW45 UP, SW46 RIGHT, SW5 2, SW6 W, SW7 S, SW8 Z, SW9 3

Commit message: Additional PCB text
Parts:
- J3: value SPACE/0 -> FIRE MAPPING
Other:
- moved on the sheet: J3
Changed lines of the file:
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@@
 	)
 	(junction
+		(at 256.54 123.19)
+		(diameter 0)
+		(color 0 0 0 0)
+	)
+	(junction
 		(at 44.45 166.37)
 		(diameter 0)
@@
 	)
 	(junction
+		(at 256.54 118.11)
+		(diameter 0)
+		(color 0 0 0 0)
+	)
+	(junction
 		(at 55.88 119.38)
 		(diameter 0)
@@
 	)
 	(junction
+		(at 256.54 120.65)
+		(diameter 0)
+		(color 0 0 0 0)
+	)
+	(junction
 		(at 66.04 128.27)
 		(diameter 0)
@@
 	(wire
 		(pts
-			(xy 259.08 120.65) (xy 247.65 120.65)
+			(xy 256.54 120.65) (xy 247.65 120.65)
 		)
 		(stroke
@@
 	(wire
 		(pts
+			(xy 256.54 118.11) (xy 259.08 118.11)
+		)
+		(stroke
+			(width 0)
+			(type default)
+		)
+	)
+	(wire
+		(pts
 			(xy 139.7 147.32) (xy 139.7 166.37)
 		)
@@
 	(wire
 		(pts
+			(xy 256.54 120.65) (xy 259.08 120.65)
+		)
+		(stroke
+			(width 0)
+			(type default)
+		)
+	)
+	(wire
+		(pts
 			(xy 247.65 91.44) (xy 247.65 120.65)
 		)
@@
 	(wire
 		(pts
+			(xy 256.54 123.19) (xy 259.08 123.19)
+		)
+		(stroke
+			(width 0)
+			(type default)
+		)
+	)
+	(wire
+		(pts
 			(xy 195.58 60.96) (xy 195.58 58.42)
 		)
@@
 	(wire
 		(pts
-			(xy 215.9 140.97) (xy 259.08 140.97)
+			(xy 215.9 140.97) (xy 256.54 140.97)
 		)
 		(stroke
@@
 	(wire
 		(pts
-			(xy 259.08 140.97) (xy 259.08 123.19)
+			(xy 256.54 140.97) (xy 256.54 123.19)
 		)
 		(stroke
@@
 	(wire
 		(pts
-			(xy 215.9 118.11) (xy 259.08 118.11)
+			(xy 215.9 118.11) (xy 256.54 118.11)
 		)
 		(stroke
@@
 	)
 	(label "FIRE_ZERO"
-		(at 259.08 118.11 180)
+		(at 256.54 118.11 180)
 		(effects
 			(font
@@
 	)
 	(label "FIRE_SPACE"
-		(at 259.08 123.19 180)
+		(at 256.54 123.19 180)
 		(effects
 			(font
@@
 	)
 	(label "FIRE"
-		(at 259.08 120.65 180)
+		(at 256.54 120.65 180)
 		(effects
 			(font
@@
 	(symbol
 		(lib_id "Connector_Generic:Conn_01x03")
-		(at 264.16 120.65 0)
+		(at 261.62 120.65 0)
 		(unit 1)
 		(body_style 1)
@@
 		(fields_autoplaced yes)
 		(property "Reference" "J3"
-			(at 266.7 119.3799 0)
+			(at 264.16 119.3799 0)
 			(show_name no)
 			(do_not_autoplace no)
@@
 			)
 		)
-		(property "Value" "SPACE/0"
-			(at 266.7 121.9199 0)
+		(property "Value" "FIRE MAPPING"
+			(at 264.16 121.9199 0)
 			(show_name no)
 			(do_not_autoplace no)
@@
 		)
 		(property "Footprint" "Connector_PinHeader_2.54mm:PinHeader_1x03_P2.54mm_Vertical"
-			(at 264.16 120.65 0)
+			(at 261.62 120.65 0)
 			(hide yes)
 			(show_name no)
@@
 		)
 		(property "Datasheet" ""
-			(at 264.16 120.65 0)
+			(at 261.62 120.65 0)
 			(hide yes)
 			(show_name no)
@@
 		)
 		(property "Description" "Generic connector, single row, 01x03, script generated (kicad-library-utils/schlib/autogen/connector/)"
-			(at 264.16 120.65 0)
+			(at 261.62 120.65 0)
 			(hide yes)
 			(show_name no)
